File: hardware/rignexo-mainboard/rignexo-mainboard.kicad_pcb (KiCad board)
At the start: 2 copper layers, 42.5 x 45 mm, 33 parts, among them J1 AudioJack3, J2 AudioJack3, K1 Relay_DPDT, Q1 MMBT3904, T1 PA0185NL, T2 PA0185NL, U2 RP2040_Zero

Commit message: Add silkscreen labels to make the board self-explanatory
Annotate connectors, volume controls, and pinouts on both sides so the
mainboard is easier to identify and use without external documentation.
Parts:
- added REF**: OSHW-Symbol_6.7x6mm_Copper, Symbol:OSHW-Symbol_6.7x6mm_Copper, B.Cu at (127.2, 129.5)
Other:
- board text added: "2.5 mm T:SPK R:PTT S:SPK"
- board text added: "3.5 mm T:PTT R:MIC S:MIC"
- board text added: "ISOLATED HAM RADIO INTERFACE"
- board text added: "MIC 3.5 mm"
- board text added: "MIC VOL"
- board text added: "RIGNEXO"
- board text added: "SPK 2.5 mm"
- board text added: "SPK VOL"
