File: hardware/rignexo-mainboard/rignexo-mainboard.kicad_pcb (KiCad board)
At the start: 2 copper layers, 42.5 x 45 mm, 34 parts, among them J1 AudioJack3, J2 AudioJack3, K1 Relay_DPDT, Q1 MMBT3904, T1 PA0185NL, T2 PA0185NL, U2 RP2040_Zero

Commit message: Fix mainboard relay coil schematic and PCB routing.
Correct the relay coil wiring error in the schematic and update the board routing; remove outdated Gerber outputs generated from the faulty layout.
Connections:
- K1 pad A1: +3.3V -> Net-(D4-A)
- K1 pad A2: Net-(D4-A) -> +3.3V
Routing:
- net +3.3V: track 67.2 -> 69.8 mm
- net Net-(D4-A): track 30.7 -> 31.4 mm, vias 0 -> 2

Commit message: Update mainboard with mode switch and local footprints.
Add a project-local CustomPartsLocal library for the 3x4mm SMD
pushbutton, wire MODE_SWITCH/MODE_LED, and add solder jumpers so
K1 lines can stay independent. Update schematic and PCB routing
to match.
Parts:
- added JP1: SolderJumper_2_Open, Jumper:SolderJumper-2_P1.3mm_Open_RoundedPad1.0x1.5mm, B.Cu at (112.7, 137.8)
- added JP2: SolderJumper_2_Open, Jumper:SolderJumper-2_P1.3mm_Open_RoundedPad1.0x1.5mm, B.Cu at (115.3, 137.8)
- added JP3: SolderJumper_2_Open, Jumper:SolderJumper-2_P1.3mm_Open_RoundedPad1.0x1.5mm, B.Cu at (126.3, 137.8)
- added JP4: SolderJumper_2_Open, Jumper:SolderJumper-2_P1.3mm_Open_RoundedPad1.0x1.5mm, B.Cu at (128.9, 137.8)
- added R13: R, Resistor_SMD:R_0805_2012Metric_Pad1.20x1.40mm_HandSolder, F.Cu at (116.5, 126.8)
- added SW1: SW_Push, CustomPartsLocal:SW_SMD_Push_3X4mm_2_pin, F.Cu at (109.8, 126.3)
- moved R12 3.01 mm to (109.8, 122.2), turned to 180 degrees
- moved R10 2.51 mm to (109.8, 119.2), turned to 180 degrees
Connections:
- J1 pad T: /PTT2 -> Net-(JP4-B)
- J2 pad R: /PTT1 -> Net-(JP1-B)
- R4 pad 1: +3.3V -> /MODE_LED
- U2 pad 18: unconnected-(U2-GPIO0-Pad18) -> /MODE_LED
- U2 pad 8: unconnected-(U2-GPIO15-Pad8) -> /MODE_SWITCH
Routing:
- net /MODE_SWITCH: track 0.00 -> 16.9 mm, vias 0 -> 2
- net Net-(JP4-B): track 0.00 -> 12.8 mm
- net GND: track 155.6 -> 166.7 mm, vias 30 -> 29
- net Net-(JP3-B): track 43.2 -> 54.2 mm
- net Net-(JP1-B): track 0.00 -> 10.9 mm
- net /PTT2: track 7.65 -> 18.5 mm, vias 0 -> 1
- net /PTT1: track 41.0 -> 30.1 mm
- net /MODE_LED: track 0.00 -> 9.04 mm
- net Net-(Q1-B): track 11.7 -> 19.9 mm
- net +3.3V: track 69.8 -> 63.7 mm, vias 4 -> 3
- net /PTT_RELAY: track 11.3 -> 6.34 mm
- net Net-(JP2-B): track 21.2 -> 22.4 mm
Other:
- board text added: "2.5 mm"
- board text added: "3.5 mm"
- board text added: "IZAR"
- board text added: "T: R:MIC S:MIC PTT"
- board text added: "T:PTT R:MIC S:MIC"
- board text added: "T:SPK R: S:SPK PTT"
- board text added: "T:SPK R:PTT S:SPK"
- board text removed: "2.5 mm T:SPK R:PTT S:SPK"
- board text removed: "3.5 mm T:PTT R:MIC S:MIC"
